File: PCBV2 - Copy/iCab.sch (KiCad schematic (older format))
At the start: 86 parts, among them J1 S5, J10 D1, J11 D2, J12 D3, J13 D4, J14 D5, J15 S5, J2 S4, J3 PGM, J4 SERIAL, J5 S3, J7 OUT, J8 S5, J9 12V, Q1 IRFZ44, Q2 IRFZ44, Q3 IRFZ44, Q4 IRFZ44, Q5 IRFZ44, SW1 SW_Push, U1 Output, U2 PIC18F2550, U3 Output, U4 L7805, Y1 Crystal

Commit message: pcb2
Parts:
- removed H1, H2: MountingHole, Mounting_Holes:MountingHole_3.2mm_M3, symbol Mechanical:MountingHole
- removed J8: S5, Terminal_Blocks:TerminalBlock_Altech_AK300-2_P5.00mm, symbol iCab-rescue:Conn_01x02
- added J6: S2, TerminalBlock_Phoenix:TerminalBlock_Phoenix_MKDS-1,5-2_1x02_P5.00mm_Horizontal, symbol Conn_01x02
- C1, C11, C12, C13, C14, C2, C4, C7, C9: footprint Capacitors_ThroughHole:CP_Radial_D5.0mm_P2.00mm -> Capacitors_THT:CP_Radial_D5.0mm_P2.00mm; symbol Device:CP1 -> CP1
- C10, C6, C8: footprint Capacitors_Tantalum_SMD:CP_Tantalum_Case-A_EIA-3216-18_Hand -> Capacitors_Tantalum_SMD:CP_Tantalum_Case-A_EIA-3216-18_Reflow; symbol Device:CP -> CP
- C3, C5: symbol Device:C -> C
- C?: renamed from C15; footprint Capacitors_ThroughHole:CP_Radial_D5.0mm_P2.00mm -> Capacitors_THT:CP_Radial_D5.0mm_P2.00mm; symbol Device:CP1 -> CP1
- D1, D4, D5, D6, D7: footprint Diodes_ThroughHole:D_T-1_P5.08mm_Horizontal -> Diodes_THT:D_T-1_P5.08mm_Horizontal; symbol Device:D -> D
- D10, D8, D9: footprint Diodes_ThroughHole:D_T-1_P5.08mm_Horizontal -> Diodes_THT:D_T-1_P10.16mm_Horizontal; symbol Device:D -> D
- D17, D2, D3: symbol Device:LED -> LED
- D?: renamed from D13; footprint Diodes_ThroughHole:D_T-1_P5.08mm_Horizontal -> Diodes_THT:D_T-1_P5.08mm_Horizontal; symbol Device:D -> D
- D?: renamed from D14; footprint Diodes_ThroughHole:D_T-1_P5.08mm_Horizontal -> Diodes_THT:D_T-1_P5.08mm_Horizontal; symbol Device:D -> D
- D?: renamed from D11; footprint Diodes_ThroughHole:D_T-1_P5.08mm_Horizontal -> Diodes_THT:D_T-1_P5.08mm_Horizontal; symbol Device:D -> D
- D?: renamed from D12; footprint Diodes_ThroughHole:D_T-1_P5.08mm_Horizontal -> Diodes_THT:D_T-1_P5.08mm_Horizontal; symbol Device:D -> D
- D?: renamed from D15; footprint Diodes_ThroughHole:D_T-1_P5.08mm_Horizontal -> Diodes_THT:D_T-1_P5.08mm_Horizontal; symbol Device:D -> D
- D?: renamed from D16; footprint Diodes_ThroughHole:D_T-1_P5.08mm_Horizontal -> Diodes_THT:D_T-1_P5.08mm_Horizontal; symbol Device:D -> D
- D?: renamed from D18; footprint Diodes_ThroughHole:D_T-1_P5.08mm_Horizontal -> Diodes_THT:D_T-1_P5.08mm_Horizontal; symbol Device:D -> D
- D?: renamed from D19; footprint Diodes_ThroughHole:D_T-1_P5.08mm_Horizontal -> Diodes_THT:D_T-1_P5.08mm_Horizontal; symbol Device:D -> D
- D?: renamed from D20; footprint Diodes_ThroughHole:D_T-1_P5.08mm_Horizontal -> Diodes_THT:D_T-1_P5.08mm_Horizontal; symbol Device:D -> D
- D?: renamed from D21; footprint Diodes_ThroughHole:D_T-1_P5.08mm_Horizontal -> Diodes_THT:D_T-1_P5.08mm_Horizontal; symbol Device:D -> D
- J1, J10, J11, J12, J13, J14, J2, J5, J9: footprint Terminal_Blocks:TerminalBlock_Altech_AK300-2_P5.00mm -> TerminalBlock_Phoenix:TerminalBlock_Phoenix_MKDS-1,5-2_1x02_P5.00mm_Horizontal; symbol iCab-rescue:Conn_01x02 -> Conn_01x02
- J3: symbol iCab-rescue:Conn_01x06 -> Conn_01x06
- J4, J7: symbol iCab-rescue:Conn_01x04 -> Conn_01x04
- J?: renamed from J15; footprint Terminal_Blocks:TerminalBlock_Altech_AK300-2_P5.00mm -> TerminalBlock_Phoenix:TerminalBlock_Phoenix_MKDS-1,5-2_1x02_P5.00mm_Horizontal; symbol iCab-rescue:Conn_01x02 -> Conn_01x02
- Q1, Q2, Q3, Q4, Q5: footprint TO_SOT_Packages_THT:TO-220-3_Vertical -> TO_SOT_Packages_THT:TO-220_Vertical; symbol iCab-rescue:IRF3205 -> IRF3205
- R1, R2, R3, R5, R6: footprint Resistors_ThroughHole:R_Axial_DIN0204_L3.6mm_D1.6mm_P7.62mm_Horizontal -> Resistors_SMD:R_0603_HandSoldering; symbol Device:R -> R
- R10, R11, R12, R13, R14, R15, R16, R17, R18, R19, R20, R21, R22, R29, R4, R7, R8, R9: symbol Device:R -> R
- SW1: footprint Buttons_Switches_ThroughHole:SW_PUSH_6mm -> Buttons_Switches_THT:SW_PUSH_6mm; symbol iCab-rescue:SW_Push -> SW_Push
- U1, U3: symbol iCab-rescue:ULN2803A -> ULN2803A
- U2: symbol iCab-rescue:PIC18F2550 -> PIC18F2550
- U4: footprint TO_SOT_Packages_THT:TO-220-3_Vertical -> TO_SOT_Packages_THT:TO-220_Vertical; symbol iCab-rescue:L7805 -> L7805
- Y1: symbol Device:Crystal -> Crystal
Connections:
- net labels added: L1, L2
- wire segments 328 -> 251
- no-connect marks 15 -> 11
Other:
- note removed: "Fuse &\nDisable"
- moved on the sheet: D2, D3, J3, J4, J7, R12, R13, R14, R15, R16, R17, R18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
